Commit message: playing around with xacro macros

File: src/arm_description/urdf/arm.urdf.xacro (robot description, xacro)
@@ -19,131 +19,173 @@
         <color rgba="0.80 0.80 0.80 1.00"/>
     </material>
-    <!-- Foot -->
-    <link name="foot">
+    <!-- Generates a box visual/collision/inertial -->
+    <xacro:macro name="prism_vci" params="side length *origin">
+        <xacro:macro name="prism_geometry">
+            <xacro:insert_block name="origin" />
+            <geometry>
+                <box size="${side} ${side} ${length}"/>
+            </geometry>
+        </xacro:macro>
         <visual>
-            <origin xyz="0 0 ${foot_length/2}" rpy="0 0 0" />
-            <geometry>
-                <box size="${link_side} ${link_side} ${foot_length}"/>
-            </geometry>
+            <xacro:prism_geometry/>
             <material name="orange"/>
         </visual>
-    </link>
-    <joint name="foot_ankle_joint" type="continuous">
-        <origin xyz="0 0 ${foot_length}" rpy="0 0 0"/>
-        <axis xyz="0 0 1" rpy="0 0 0"/>
-        <parent link="foot"/>
-        <child link="ankle"/>
-    </joint>
-    <!-- Ankle -->
-    <link name="ankle">
+        <collision>
+            <xacro:prism_geometry/>
+        </collision>
+    </xacro:macro>
+    <!-- Generates a cylinder visual/collision/inertial -->
+    <xacro:macro name="cylinder_vci" params="radius length *origin">
+        <xacro:macro name="cylinder_geometry">
+            <xacro:insert_block name="origin" />
+            <geometry>
+                <cylinder length ="${length}" radius="${radius}"/>
+            </geometry>
+        </xacro:macro>
         <visual>
-            <origin xyz="0 0 ${ankle_length/2}" rpy="0 0 0" />
-            <geometry>
-                <box size="${link_side} ${link_side} ${ankle_length}"/>
-            </geometry>
-            <material name="orange"/>
-        </visual>
-        <visual>
-            <origin xyz="0 0 0" rpy="0 0 0" />
-            <geometry>
-                <cylinder length ="${joint_length}" radius="${joint_radius}"/>
-            </geometry>
+            <xacro:cylinder_geometry/>
             <material name="gray"/>
         </visual>
+        <collision>
+            <xacro:cylinder_geometry/>
+        </collision>
+    </xacro:macro>
+    <!-- Generates child joint of parent -->
+    <xacro:macro name="arm_joint" params="name parent dist:=0 type axis">
+        <joint name="${parent}_${name}_joint" type="continuous">
+            <origin xyz="0 0 ${dist}" rpy="0 0 0"/>
+            <parent link="${parent}"/>
+            <child link="${name}"/>
+            <axis xyz="${axis}" />
+        </joint>
+        <link name="${parent}">
+            <xacro:prism_vci length="${dist}" side="${link_side}">
+                <origin xyz="0 0 ${dist/2}" rpy="0 0 0"/>
+            </xacro:prism_vci>
+            <xacro:if value="${type!='fixed'}">
+                <xacro:cylinder_vci radius="${joint_radius}" length="${joint_length}">
+                    <xacro:if value="${axis=='0 0 1'}">
+                        <origin xyz="0 0 ${dist}" rpy="0 0 0"/>
+                    </xacro:if>
+                    <xacro:if value="${axis!='0 0 1'}">
+                        <origin xyz="0 0 ${dist}" rpy="${PI/2} 0 0"/>
+                    </xacro:if>
+                </xacro:cylinder_vci>
+            </xacro:if>
+        </link>
+    </xacro:macro>
+    <!-- World frame (for Gazebo) -->
+    <link name="world" />
+    <!-- Arm fixed to world frame  -->
+    <joint name="world_foot_joint" type="fixed">
+        <parent link="world"/>
+        <child link="foot"/>
+    </joint>
+    <!-- Joints Chain -->
+    <xacro:arm_joint name="ankle" parent="foot"  type="continuous" axis="0 0 1" dist="${foot_length}"  />
+    <xacro:arm_joint name="leg"   parent="ankle" type="continuous" axis="1 0 0" dist="${ankle_length}" />
+    <xacro:arm_joint name="arm"   parent="leg"   type="continuous" axis="1 0 0" dist="${leg_length}"   />
+    <xacro:arm_joint name="wrist" parent="arm"   type="continuous" axis="0 0 1" dist="${arm_length}"   />
+    <xacro:arm_joint name="hand"  parent="wrist" type="continuous" axis="1 0 0" dist="${wrist_length}" />
+    <!-- End effector -->
+    <link name="hand">
+        <xacro:prism_vci length="${hand_length}" side="${link_side}">
+            <origin xyz="0 0 ${hand_length/2}" rpy="0 0 0"/>
+        </xacro:prism_vci>
     </link>
-    <joint name="ankle_leg_joint" type="revolute">
-        <origin xyz="0 0 ${ankle_length}" rpy="0 -${PI/2} 0"/>
-        <axis xyz="0 0 1" rpy="0 0 0"/>
-        <limit effort="30" velocity="1.0" lower="${-PI/2}" upper="${PI/2}" />
-        <parent link="ankle"/>
-        <child link="leg"/>
-    </joint>
-    <!-- Leg -->
-    <link name="leg">
-        <visual>
-            <origin xyz="${leg_length/2} 0 0" rpy="0 0 0" />
-            <geometry>
-                <box size="${leg_length} ${link_side} ${link_side}"/>
-            </geometry>
-            <material name="orange"/>
-        </visual>
-        <visual>
-            <origin xyz="0 0 0" rpy="0 0 0" />
-            <geometry>
-                <cylinder length ="${joint_length}" radius="${joint_radius}"/>
-            </geometry>
-            <material name="gray"/>
-        </visual>
-    </link>
-    <joint name="leg_arm_joint" type="revolute">
-        <origin xyz="${leg_length} 0 0" rpy="0 0 0"/>
-        <axis xyz="0 0 1" rpy="0 0 0"/>
-        <limit effort="30" velocity="1.0" lower="${-2*PI/3}" upper="${2*PI/3}" />
-        <parent link="leg"/>
-        <child link="arm"/>
-    </joint>
-    <!-- Arm -->
-    <link name="arm">
-        <visual>
-            <origin xyz="${arm_length/2} 0 0" rpy="0 0 0" />
-            <geometry>
-                <box size="${arm_length} ${link_side} ${link_side}"/>
-            </geometry>
-            <material name="orange"/>
-        </visual>
-        <visual>
-            <origin xyz="0 0 0" rpy="0 0 0" />
-            <geometry>
-                <cylinder length ="${joint_length}" radius="${joint_radius}"/>
-            </geometry>
-            <material name="gray"/>
-        </visual>
-    </link>
-    <joint name="arm_wrist_joint" type="continuous">
-        <origin xyz="${arm_length} 0 0" rpy="0 ${PI/2} 0"/>
-        <axis xyz="0 0 1" rpy="0 0 0"/>
-        <parent link="arm"/>
-        <child link="wrist"/>
-    </joint>
-    <!-- Wrist -->
-    <link name="wrist">
-        <visual>
-            <origin xyz="0 0 ${wrist_length/2}" rpy="0 0 0" />
-            <geometry>
-                <box size="${link_side} ${link_side} ${wrist_length}"/>
-            </geometry>
-            <material name="orange"/>
-        </visual>
-        <visual>
-            <origin xyz="0 0 0" rpy="0 0 0" />
-            <geometry>
-                <cylinder length ="${joint_length}" radius="${joint_radius}"/>
-            </geometry>
-            <material name="gray"/>
-        </visual>
-    </link>
-    <joint name="wrist_hand_joint" type="revolute">
-        <origin xyz="0 0 ${wrist_length}" rpy="0 ${-PI/2} 0"/>
-        <axis xyz="0 0 1" rpy="0 0 0"/>
-        <limit effort="30" velocity="1.0" lower="${-PI/2}" upper="${PI/2}" />
-        <parent link="wrist"/>
-        <child link="hand"/>
-    </joint>
-    <!-- Hand -->
-    <link name="hand">
-        <visual>
-            <origin xyz="${hand_length/2} 0 0" rpy="0 0 0" />
-            <geometry>
-                <box size="${wrist_length} ${link_side} ${link_side}"/>
-            </geometry>
-            <material name="orange"/>
-        </visual>
-        <visual>
-            <origin xyz="0 0 0" rpy="0 0 0" />
-            <geometry>
-                <cylinder length ="${joint_length}" radius="${joint_radius}"/>
-            </geometry>
-            <material name="gray"/>
-        </visual>
-    </link>
+    <!--&lt;!&ndash; Ankle &ndash;&gt;-->
+    <!--<xacro:arm_link name="ankle" length="${ankle_length}">-->
+        <!--<origin xyz="0 0 ${ankle_length/2}" rpy="0 0 0" />-->
+    <!--</xacro:arm_link>-->
+    <!--<joint name="ankle_leg_joint" type="revolute">-->
+        <!--<origin xyz="0 0 ${ankle_length}" rpy="0 -${PI/2} 0"/>-->
+        <!--<axis xyz="0 0 1" rpy="0 0 0"/>-->
+        <!--<limit effort="30" velocity="1.0" lower="${-PI/2}" upper="${PI/2}" />-->
+        <!--<parent link="ankle"/>-->
+        <!--<child link="leg"/>-->
+    <!--</joint>-->
+    <!--&lt;!&ndash; Leg &ndash;&gt;-->
+    <!--<link name="leg">-->
+        <!--<visual>-->
+            <!--<origin xyz="${leg_length/2} 0 0" rpy="0 0 0" />-->
+            <!--<geometry>-->
+                <!--<box size="${leg_length} ${link_side} ${link_side}"/>-->
+            <!--</geometry>-->
+            <!--<material name="orange"/>-->
+        <!--</visual>-->
+        <!--<visual>-->
+            <!--<geometry>-->
+                <!--<cylinder length ="${joint_length}" radius="${joint_radius}"/>-->
+            <!--</geometry>-->
+            <!--<material name="gray"/>-->
+        <!--</visual>-->
+    <!--</link>-->
+    <!--<joint name="leg_arm_joint" type="revolute">-->
+        <!--<origin xyz="${leg_length} 0 0" rpy="0 0 0"/>-->
+        <!--<axis xyz="0 0 1" rpy="0 0 0"/>-->
+        <!--<limit effort="30" velocity="1.0" lower="${-2*PI/3}" upper="${2*PI/3}" />-->
+        <!--<parent link="leg"/>-->
+        <!--<child link="arm"/>-->
+    <!--</joint>-->
+    <!--&lt;!&ndash; Arm &ndash;&gt;-->
+    <!--<link name="arm">-->
+        <!--<visual>-->
+            <!--<origin xyz="${arm_length/2} 0 0" rpy="0 0 0" />-->
+            <!--<geometry>-->
+                <!--<box size="${arm_length} ${link_side} ${link_side}"/>-->
+            <!--</geometry>-->
+            <!--<material name="orange"/>-->
+        <!--</visual>-->
+        <!--<visual>-->
+            <!--<geometry>-->
+                <!--<cylinder length ="${joint_length}" radius="${joint_radius}"/>-->
+            <!--</geometry>-->
+            <!--<material name="gray"/>-->
+        <!--</visual>-->
+    <!--</link>-->
+    <!--<joint name="arm_wrist_joint" type="continuous">-->
+        <!--<origin xyz="${arm_length} 0 0" rpy="0 ${PI/2} 0"/>-->
+        <!--<axis xyz="0 0 1" rpy="0 0 0"/>-->
+        <!--<parent link="arm"/>-->
+        <!--<child link="wrist"/>-->
+    <!--</joint>-->
+    <!--&lt;!&ndash; Wrist &ndash;&gt;-->
+    <!--<link name="wrist">-->
+        <!--<visual>-->
+            <!--<origin xyz="0 0 ${wrist_length/2}" rpy="0 0 0" />-->
+            <!--<geometry>-->
+                <!--<box size="${link_side} ${link_side} ${wrist_length}"/>-->
+            <!--</geometry>-->
+            <!--<material name="orange"/>-->
+        <!--</visual>-->
+        <!--<visual>-->
+            <!--<geometry>-->
+                <!--<cylinder length ="${joint_length}" radius="${joint_radius}"/>-->
+            <!--</geometry>-->
+            <!--<material name="gray"/>-->
+        <!--</visual>-->
+    <!--</link>-->
+    <!--<joint name="wrist_hand_joint" type="revolute">-->
+        <!--<origin xyz="0 0 ${wrist_length}" rpy="0 ${-PI/2} 0"/>-->
+        <!--<axis xyz="0 0 1" rpy="0 0 0"/>-->
+        <!--<limit effort="30" velocity="1.0" lower="${-PI/2}" upper="${PI/2}" />-->
+        <!--<parent link="wrist"/>-->
+        <!--<child link="hand"/>-->
+    <!--</joint>-->
+    <!--&lt;!&ndash; Hand &ndash;&gt;-->
+    <!--<link name="hand">-->
+        <!--<visual>-->
+            <!--<origin xyz="${hand_length/2} 0 0" rpy="0 0 0" />-->
+            <!--<geometry>-->
+                <!--<box size="${wrist_length} ${link_side} ${link_side}"/>-->
+            <!--</geometry>-->
+            <!--<material name="orange"/>-->
+        <!--</visual>-->
+        <!--<visual>-->
+            <!--<geometry>-->
+                <!--<cylinder length ="${joint_length}" radius="${joint_radius}"/>-->
+            <!--</geometry>-->
+            <!--<material name="gray"/>-->
+        <!--</visual>-->
+    <!--</link>-->
 </robot>
